File: Kicad/Northstart Floating point.kicad_sch (KiCad schematic)
At the start: 83 parts, among them J12 Jumper_2_Open, J13 Jumper_2_Open, J14 Jumper_2_Open, J3 S100_conn, Y1 Crystal

Commit message: Add files via upload
Parts:
- renumbered D1 to D_RAM1, L1 to L_RAM1
Connections:
- net GND: now also L_RAM1.8 (GND), MPXR1.8 (GND)
- net VCC: now also L_RAM1.16 (VCC), MPXR1.16 (VCC)
- no-connect marks 0 -> 59
Other:
- moved on the sheet: AOI1B, NR1D, OC1B, ST1D
